File: pcb/atlas-11.kicad_pcb (KiCad board)
At the start: 2 copper layers, 115.2 x 61.7 mm, 5 parts, among them J1 USB_C_Receptacle, J2 DCJ-11 SBC Expansion Bus, J3 Micro_SD_Card_Det2, U1 RP2350B-QFN80, U2 TPS22810DBVR

Commit message: add more sections from rp2350 minimal example
Parts:
- added C1: 10u, Capacitor_SMD:C_0805_2012Metric, F.Cu at (133.0, 71.7)
- added C2: 100n, Capacitor_SMD:C_0402_1005Metric, F.Cu at (129.1, 61.6)
- added C3: 15p, Capacitor_SMD:C_0402_1005Metric, F.Cu at (129.1, 63.6)
- added C4: 15p, Capacitor_SMD:C_0402_1005Metric, F.Cu at (129.1, 65.6)
- added C5: 10u, Capacitor_SMD:C_0805_2012Metric, F.Cu at (133.0, 74.7)
- added R1: DNF, Resistor_SMD:R_0402_1005Metric, F.Cu at (119.5, 61.7)
- added R10: 0, Resistor_SMD:R_0402_1005Metric, F.Cu at (119.5, 71.6)
- added R2: 1k, Resistor_SMD:R_0402_1005Metric, F.Cu at (119.5, 63.6)
- added R4: 1k, Resistor_SMD:R_0402_1005Metric, F.Cu at (119.5, 65.6)
- added R6: 1k, Resistor_SMD:R_0402_1005Metric, F.Cu at (119.5, 67.6)
- added R9: DNF, Resistor_SMD:R_0402_1005Metric, F.Cu at (119.5, 69.6)
- added SW1: SW_Push, Button_Switch_SMD:SW_Push_1P1T_NO_Vertical_Wuerth_434133025816, F.Cu at (124.3, 63.0)
- added SW2: SW_Push, Button_Switch_SMD:SW_Push_1P1T_NO_Vertical_Wuerth_434133025816, F.Cu at (124.3, 67.8)
- added U4: NCP1117-3.3_SOT223, Package_TO_SOT_SMD:SOT-223-3_TabPin2, F.Cu at (125.9, 74.4)
- added Y1: ABM8-272-T3, Crystal:Crystal_SMD_3225-4Pin_3.2x2.5mm, F.Cu at (133.2, 62.9)

Commit message: schematics & pcb work
Parts:
- added C10: 4.7u, Capacitor_SMD:C_0402_1005Metric, F.Cu at (121.3, 93.3)
- added C11: 100n, Capacitor_SMD:C_0402_1005Metric, F.Cu at (121.3, 95.3)
- added C12: 100n, Capacitor_SMD:C_0402_1005Metric, F.Cu at (121.3, 97.2)
- added C13: 100n, Capacitor_SMD:C_0402_1005Metric, F.Cu at (124.2, 89.4)
- added C14: 100n, Capacitor_SMD:C_0402_1005Metric, F.Cu at (124.2, 91.3)
- added C15: 100n, Capacitor_SMD:C_0402_1005Metric, F.Cu at (124.2, 93.3)
- added C16: 100n, Capacitor_SMD:C_0402_1005Metric, F.Cu at (124.2, 95.3)
- added C17: 100n, Capacitor_SMD:C_0402_1005Metric, F.Cu at (124.2, 97.2)
- added C18: 100n, Capacitor_SMD:C_0402_1005Metric, F.Cu at (127.0, 89.4)
- added C19: 100n, Capacitor_SMD:C_0402_1005Metric, F.Cu at (127.0, 91.3)
- added C20: 100n, Capacitor_SMD:C_0402_1005Metric, F.Cu at (127.0, 93.3)
- added C8: 100n, Capacitor_SMD:C_0402_1005Metric, F.Cu at (121.3, 89.4)
- added C9: 4.7u, Capacitor_SMD:C_0402_1005Metric, F.Cu at (121.3, 91.3)
- added J4: DCJ-11 SBC Bus Probe Interface, Library:DCJ-11 SBC Expansion Port Debug Header, F.Cu at (75.2, 97.2)
- added R5: 33, Resistor_SMD:R_0402_1005Metric, F.Cu at (129.9, 89.4)
- added R7: 27, Resistor_SMD:R_0402_1005Metric, F.Cu at (129.9, 91.4)
- added R8: 27, Resistor_SMD:R_0402_1005Metric, F.Cu at (129.9, 93.3)
- J1: value USB_C_Receptacle -> USB
- moved U2 8.64 mm to (92.0, 84.9)
- moved U1 4.55 mm to (58.1, 83.3)
Connections:
- J2 pad 10: /DAL6 -> DAL6
- J2 pad 11: /DAL0 -> DAL0
- J2 pad 25: VCC -> SBC_POWER
- J2 pad 4: /DAL1 -> DAL1
- J2 pad 40: /DAL7 -> DAL7
- J2 pad 41: /DAL5 -> DAL5
- J2 pad 42: /DAL12 -> DAL12
- J2 pad 43: /DAL11 -> DAL11
- J2 pad 44: /DAL13 -> DAL13
- J2 pad 45: /DAL10 -> DAL10
- J2 pad 46: /DAL2 -> DAL2
- J2 pad 47: /DAL8 -> DAL8
- J2 pad 5: /DAL3 -> DAL3
- J2 pad 6: /DAL15 -> DAL15
- J2 pad 7: /DAL14 -> DAL14
- J2 pad 8: /DAL9 -> DAL9
- J2 pad 9: /DAL4 -> DAL4
- R1 pad 2: /FLASH_SS -> /QSPI_SS
- R6 pad 1: unconnected-(R6-Pad1) -> /QSPI_SS
- SW2 pad 2: unconnected-(SW2-Pad2) -> Net-(U1-RUN)
- U1 pad 10: unconnected-(U1-DVDD-Pad10) -> +1V1
- U1 pad 11: unconnected-(U1-GPIO12-Pad11) -> DAL7
- U1 pad 12: unconnected-(U1-GPIO13-Pad12) -> DAL8
- U1 pad 13: unconnected-(U1-GPIO14-Pad13) -> DAL9
- U1 pad 14: unconnected-(U1-GPIO15-Pad14) -> DAL10
- U1 pad 15: unconnected-(U1-IOVDD-Pad15) -> +3V3
- U1 pad 16: unconnected-(U1-GPIO16-Pad16) -> DAL11
- U1 pad 17: unconnected-(U1-GPIO17-Pad17) -> DAL12
- U1 pad 18: unconnected-(U1-GPIO18-Pad18) -> DAL13
- U1 pad 19: unconnected-(U1-GPIO19-Pad19) -> DAL14
- U1 pad 2: unconnected-(U1-GPIO5-Pad2) -> DAL0
- U1 pad 20: unconnected-(U1-GPIO20-Pad20) -> DAL15
- U1 pad 24: unconnected-(U1-IOVDD-Pad24) -> +3V3
- U1 pad 29: unconnected-(U1-IOVDD-Pad29) -> +3V3
- U1 pad 3: unconnected-(U1-GPIO6-Pad3) -> DAL1
- U1 pad 30: unconnected-(U1-XIN-Pad30) -> /XIN
- U1 pad 31: unconnected-(U1-XOUT-Pad31) -> /XOUT
- U1 pad 32: unconnected-(U1-DVDD-Pad32) -> +1V1
- U1 pad 35: unconnected-(U1-RUN-Pad35) -> Net-(U1-RUN)
- U1 pad 4: unconnected-(U1-GPIO7-Pad4) -> DAL2
- U1 pad 41: unconnected-(U1-IOVDD-Pad41) -> +3V3
- U1 pad 5: unconnected-(U1-IOVDD-Pad5) -> +3V3
- U1 pad 50: unconnected-(U1-IOVDD-Pad50) -> +3V3
- U1 pad 51: unconnected-(U1-DVDD-Pad51) -> +1V1
- U1 pad 59: unconnected-(U1-ADC_AVDD-Pad59) -> +3V3
- U1 pad 6: unconnected-(U1-GPIO8-Pad6) -> DAL3
- U1 pad 60: unconnected-(U1-IOVDD-Pad60) -> +3V3
- U1 pad 61: unconnected-(U1-VREG_AVDD-Pad61) -> /VREG_AVDD
- U1 pad 62: unconnected-(U1-VREG_PGND-Pad62) -> GND
- U1 pad 63: unconnected-(U1-VREG_LX-Pad63) -> /VREG_LX
- U1 pad 64: unconnected-(U1-VREG_VIN-Pad64) -> +3V3
- U1 pad 65: unconnected-(U1-VREG_FB-Pad65) -> +1V1
- U1 pad 66: unconnected-(U1-USB_DM-Pad66) -> Net-(U1-USB_DM)
- U1 pad 67: unconnected-(U1-USB_DP-Pad67) -> Net-(U1-USB_DP)
- U1 pad 68: unconnected-(U1-USB_OTP_VDD-Pad68) -> +3V3
- U1 pad 69: unconnected-(U1-QSPI_IOVDD-Pad69) -> +3V3
- U1 pad 7: unconnected-(U1-GPIO9-Pad7) -> DAL4
- U1 pad 70: unconnected-(U1-QSPI_SD3-Pad70) -> /QSPI_SD3
- U1 pad 71: unconnected-(U1-QSPI_SCLK-Pad71) -> /QSPI_SCLK
- U1 pad 72: unconnected-(U1-QSPI_SD0-Pad72) -> /QSPI_SD0
- U1 pad 73: unconnected-(U1-QSPI_SD2-Pad73) -> /QSPI_SD2
- U1 pad 74: unconnected-(U1-QSPI_SD1-Pad74) -> /QSPI_SD1
- U1 pad 75: unconnected-(U1-QSPI_SS-Pad75) -> /QSPI_SS
- U1 pad 76: unconnected-(U1-IOVDD-Pad76) -> +3V3
- U1 pad 79: unconnected-(U1-GPIO2-Pad79) -> SBC_ON
- U1 pad 8: unconnected-(U1-GPIO10-Pad8) -> DAL5
- U1 pad 9: unconnected-(U1-GPIO11-Pad9) -> DAL6
- U2 pad 1: unconnected-(U2-VOUT-Pad1) -> SBC_POWER
- U2 pad 4: Net-(U2-GND-Pad4) -> GND
- U2 pad 5: unconnected-(U2-EN/UVLO-Pad5) -> SBC_ON
- U2 pad 6: unconnected-(U2-VIN-Pad6) -> VBUS

Commit message: fix tps22810 pinout
Parts:
- C20: value 100n -> 1µ
Connections:
- U2 pad 1: SBC_POWER -> VBUS
- U2 pad 2: unconnected-(U2-QOD-Pad2) -> GND
- U2 pad 3: unconnected-(U2-CT-Pad3) -> SBC_ON
- U2 pad 4: GND -> unconnected-(U2-CT-Pad4)
- U2 pad 5: SBC_ON -> unconnected-(U2-QOD-Pad5)
- U2 pad 6: VBUS -> SBC_POWER
Changed lines of the file:
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@@
 	(net 97 "unconnected-(U1-GPIO28-Pad36)")
 	(net 98 "unconnected-(U1-GPIO25-Pad26)")
-	(net 99 "unconnected-(U2-CT-Pad3)")
-	(net 100 "unconnected-(U2-QOD-Pad2)")
+	(net 99 "unconnected-(U2-CT-Pad4)")
+	(net 100 "unconnected-(U2-QOD-Pad5)")
 	(net 101 "VBUS")
 	(net 102 "+3V3")
@@
 			)
 		)
-		(property "Value" "100n"
+		(property "Value" "1µ"
 			(at 0 1.16 0)
 			(layer "F.Fab")
@@
 			(layers "F.Cu" "F.Mask" "F.Paste")
 			(roundrect_rratio 0.25)
+			(net 101 "VBUS")
+			(pinfunction "VIN")
+			(pintype "power_in")
+		)
+		(pad "2" smd roundrect
+			(at -1.35 0)
+			(size 1.56 0.65)
+			(layers "F.Cu" "F.Mask" "F.Paste")
+			(roundrect_rratio 0.25)
+			(net 29 "GND")
+			(pinfunction "GND")
+			(pintype "power_in")
+		)
+		(pad "3" smd roundrect
+			(at -1.35 0.95)
+			(size 1.56 0.65)
+			(layers "F.Cu" "F.Mask" "F.Paste")
+			(roundrect_rratio 0.25)
+			(net 62 "SBC_ON")
+			(pinfunction "EN/UVLO")
+			(pintype "input")
+		)
+		(pad "4" smd roundrect
+			(at 1.35 0.95)
+			(size 1.56 0.65)
+			(layers "F.Cu" "F.Mask" "F.Paste")
+			(roundrect_rratio 0.25)
+			(net 99 "unconnected-(U2-CT-Pad4)")
+			(pinfunction "CT")
+			(pintype "output+no_connect")
+		)
+		(pad "5" smd roundrect
+			(at 1.35 0)
+			(size 1.56 0.65)
+			(layers "F.Cu" "F.Mask" "F.Paste")
+			(roundrect_rratio 0.25)
+			(net 100 "unconnected-(U2-QOD-Pad5)")
+			(pinfunction "QOD")
+			(pintype "open_collector+no_connect")
+		)
+		(pad "6" smd roundrect
+			(at 1.35 -0.95)
+			(size 1.56 0.65)
+			(layers "F.Cu" "F.Mask" "F.Paste")
+			(roundrect_rratio 0.25)
 			(net 8 "SBC_POWER")
 			(pinfunction "VOUT")
 			(pintype "power_out")
 		)
-		(pad "2" smd roundrect
-			(at -1.35 0)
-			(size 1.56 0.65)
-			(layers "F.Cu" "F.Mask" "F.Paste")
-			(roundrect_rratio 0.25)
-			(net 100 "unconnected-(U2-QOD-Pad2)")
-			(pinfunction "QOD")
-			(pintype "open_collector+no_connect")
-		)
-		(pad "3" smd roundrect
-			(at -1.35 0.95)
-			(size 1.56 0.65)
-			(layers "F.Cu" "F.Mask" "F.Paste")
-			(roundrect_rratio 0.25)
-			(net 99 "unconnected-(U2-CT-Pad3)")
-			(pinfunction "CT")
-			(pintype "output+no_connect")
-		)
-		(pad "4" smd roundrect
-			(at 1.35 0.95)
-			(size 1.56 0.65)
-			(layers "F.Cu" "F.Mask" "F.Paste")
-			(roundrect_rratio 0.25)
-			(net 29 "GND")
-			(pinfunction "GND")
-			(pintype "power_in")
-		)
-		(pad "5" smd roundrect
-			(at 1.35 0)
-			(size 1.56 0.65)
-			(layers "F.Cu" "F.Mask" "F.Paste")
-			(roundrect_rratio 0.25)
-			(net 62 "SBC_ON")
-			(pinfunction "EN/UVLO")
-			(pintype "input")
-		)
-		(pad "6" smd roundrect
-			(at 1.35 -0.95)
-			(size 1.56 0.65)
-			(layers "F.Cu" "F.Mask" "F.Paste")
-			(roundrect_rratio 0.25)
-			(net 101 "VBUS")
-			(pinfunction "VIN")
-			(pintype "power_in")
-		)
 		(embedded_fonts no)

Commit message: pcb work
Parts:
- removed J3: Micro_SD_Card_Det2, Connector_USB:USB_C_Plug_JAE_DX07P024AJ1
- added P1: USB, Connector_USB:USB_C_Receptacle_G-Switch_GT-USB-7010ASV, F.Cu at (36.7, 83.1)
- C10, C11, C12, C13, C14, C15, C16, C17, C18, C19, C2, C20, C3, C4, C8, C9: footprint Capacitor_SMD:C_0402_1005Metric -> Capacitor_SMD:C_0603_1608Metric_Pad1.08x0.95mm_HandSolder
- J1: value USB -> Micro_SD_Card_Det1; footprint Connector_Card:microSD_HC_Hirose_DM3AT-SF-PEJM5 -> Connector_Card:microSD_HC_Hirose_DM3BT-DSF-PEJS
- R1, R10, R2, R4, R5, R6, R7, R8, R9: footprint Resistor_SMD:R_0402_1005Metric -> Resistor_SMD:R_0603_1608Metric_Pad0.98x0.95mm_HandSolder
- SW1: value SW_Push -> USB BOOT
- SW2: value SW_Push -> RUN
- moved C13 110.3 mm to (13.9, 87.6)
- moved C14 110.3 mm to (13.9, 89.6)
- moved C15 110.3 mm to (13.9, 91.5)
- moved C16 110.3 mm to (13.9, 93.5)
- moved C17 110.3 mm to (13.9, 95.5)
- moved C2 110.3 mm to (18.9, 59.9)
- moved R5 110.3 mm to (19.7, 87.6)
- moved R7 110.3 mm to (19.7, 89.6)
- moved R8 110.3 mm to (19.7, 91.6)
- moved C1 110.3 mm to (22.8, 69.9)
- moved C10 110.3 mm to (11.0, 91.5)
- moved C11 110.3 mm to (11.0, 93.5)
- moved C12 110.3 mm to (11.0, 95.5)
- moved C18 110.3 mm to (16.8, 87.6)
- moved C19 110.3 mm to (16.8, 89.6)
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Connections:
- net /~{USB_BOOT} renamed Net-(R6-Pad2)
- J1 pad 1: (no net) -> unconnected-(J1-DAT2-Pad1)
- J1 pad 10: (no net) -> unconnected-(J1-SHIELD-Pad10)
- J1 pad 2: (no net) -> SDCARD_CS
- J1 pad 3: (no net) -> SDCARD_MOSI
- J1 pad 4: (no net) -> +3V3
- J1 pad 5: (no net) -> SDCARD_CLK
- J1 pad 6: (no net) -> GND
- J1 pad 7: (no net) -> SDCARD_MISO
- J1 pad 8: (no net) -> unconnected-(J1-DAT1-Pad8)
- J1 pad 9: (no net) -> SDCARD_DET
- J2 pad 13: /HALT -> HALT
- J2 pad 15: /~{BUFCTL} -> ~{BUFCTL}
- J2 pad 17: /~{CONT} -> ~{CONT}
- J2 pad 21: /INIT -> INIT
- J2 pad 34: /~{SCTL} -> ~{SCTL}
- J2 pad 35: /~{ALE} -> ~{ALE}
- J2 pad 48: /~{IO} -> ~{IO}
- J4 pad 13: /HALT -> HALT
- J4 pad 15: /~{BUFCTL} -> ~{BUFCTL}
- J4 pad 17: /~{CONT} -> ~{CONT}
- J4 pad 21: /INIT -> INIT
- J4 pad 34: /~{SCTL} -> ~{SCTL}
- J4 pad 35: /~{ALE} -> ~{ALE}
- J4 pad 48: /~{IO} -> ~{IO}
- R4 pad 1: Net-(R4-Pad1) -> Net-(U1-RUN)
- R4 pad 2: GND -> Net-(R4-Pad2)
- SW2 pad 1: Net-(R4-Pad1) -> GND
- SW2 pad 2: Net-(U1-RUN) -> Net-(R4-Pad2)
- U1 pad 21: unconnected-(U1-GPIO21-Pad21) -> ~{BUFCTL}
- U1 pad 22: unconnected-(U1-GPIO22-Pad22) -> HALT
- U1 pad 23: unconnected-(U1-GPIO23-Pad23) -> ~{ALE}
- U1 pad 25: unconnected-(U1-GPIO24-Pad25) -> ~{SCTL}
- U1 pad 26: unconnected-(U1-GPIO25-Pad26) -> ~{CONT}
- U1 pad 27: unconnected-(U1-GPIO26-Pad27) -> INIT
- U1 pad 28: unconnected-(U1-GPIO27-Pad28) -> ~{IO}
- U1 pad 33: unconnected-(U1-SWCLK-Pad33) -> /SWCLK
- U1 pad 34: unconnected-(U1-SWDIO-Pad34) -> /SWDIO
- U1 pad 53: unconnected-(U1-GPIO42_ADC2-Pad53) -> SDCARD_DET
- U1 pad 54: unconnected-(U1-GPIO43_ADC3-Pad54) -> SDCARD_MOSI
- U1 pad 55: unconnected-(U1-GPIO44_ADC4-Pad55) -> SDCARD_MISO
- U1 pad 56: unconnected-(U1-GPIO45_ADC5-Pad56) -> SDCARD_CS
- U1 pad 57: unconnected-(U1-GPIO46_ADC6-Pad57) -> SDCARD_CLK
- U1 pad 77: unconnected-(U1-GPIO0-Pad77) -> UART0_TX
- U1 pad 78: unconnected-(U1-GPIO1-Pad78) -> UART0_RX
- U1 pad 81: unconnected-(U1-GND-Pad81) -> GND
Other:
- board size 115.2 x 61.7 mm -> 121.5 x 70.7 mm

Commit message: pcb work
Parts:
- removed R1, R9: DNF, Resistor_SMD:R_0603_1608Metric_Pad0.98x0.95mm_HandSolder
- removed R10: 0, Resistor_SMD:R_0603_1608Metric_Pad0.98x0.95mm_HandSolder
- added C21: 4.7µ, Capacitor_SMD:C_0603_1608Metric_Pad1.08x0.95mm_HandSolder, F.Cu at (50.8, 69.1)
- added C7: 4.7µ, Capacitor_SMD:C_0603_1608Metric_Pad1.08x0.95mm_HandSolder, F.Cu at (49.1, 72.3)
- added J3: SWD, Connector_PinHeader_2.54mm:PinHeader_1x03_P2.54mm_Horizontal, F.Cu at (35.3, 56.1)
- added J5: UART0, Connector_PinSocket_2.54mm:PinSocket_1x03_P2.54mm_Horizontal, F.Cu at (51.7, 56.1)
- added J6: User Port, Connector_PinHeader_2.54mm:PinHeader_2x09_P2.54mm_Vertical, F.Cu at (84.6, 78.7)
- added J7: Pico Bits, Connector_PinHeader_2.54mm:PinHeader_2x09_P2.54mm_Vertical, F.Cu at (84.7, 86.0)
- added L1: 3.3µ, Inductor_SMD:L_0805_2012Metric_Pad1.15x1.40mm_HandSolder, F.Cu at (52.9, 72.0)
- added U3: W25Q128JVS, Package_SO:SOIC-8_5.3x5.3mm_P1.27mm, F.Cu at (46.9, 79.9)
- added U5: MCP23017, Package_SO:SOIC-28W_7.5x17.9mm_P1.27mm, F.Cu at (97.4, 67.5)
- added U6: MCP23017_SO, Package_SO:SOIC-28W_7.5x17.9mm_P1.27mm, F.Cu at (97.5, 53.1)
- C9: value 4.7u -> 4.7µ
- J1: value Micro_SD_Card_Det1 -> SD Card
- SW1: value USB BOOT -> BOOTSEL
- U1: value RP2350B-QFN80 -> RP2350B
- U4: value NCP1117-3.3_SOT223 -> NCP1117-3.3
- moved R4 73.7 mm to (82.1, 52.7), turned to 180 degrees
- moved SW2 69.9 mm to (82.1, 49.7)
- moved R6 67.7 mm to (75.7, 52.7), turned to 180 degrees
- moved SW1 62.6 mm to (75.6, 49.8)
- moved C10 59.5 mm to (67.9, 74.0), turned to 90 degrees
- moved C17 58.0 mm to (64.7, 67.6), turned to 90 degrees
- moved C12 58.0 mm to (61.8, 67.6), turned to 90 degrees
- moved U2 55.7 mm to (37.5, 96.1), turned to 90 degrees
- moved C8 53.1 mm to (60.2, 67.6), turned to 90 degrees
- moved C11 50.6 mm to (60.7, 83.7), turned to -90 degrees
- moved C16 50.5 mm to (57.3, 67.6), turned to 90 degrees
- moved C9 47.7 mm to (54.1, 69.1), turned to 90 degrees
- moved C18 46.2 mm to (62.8, 83.7), turned to -90 degrees
- moved C13 45.0 mm to (58.8, 83.7), turned to -90 degrees
- moved C15 42.5 mm to (53.0, 74.8), turned to 180 degrees
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Connections:
- U1 pad 1: unconnected-(U1-GPIO4-Pad1) -> LED1
- U1 pad 36: unconnected-(U1-GPIO28-Pad36) -> GPIO28
- U1 pad 37: unconnected-(U1-GPIO29-Pad37) -> GPIO29
- U1 pad 38: unconnected-(U1-GPIO30-Pad38) -> GPIO30
- U1 pad 39: unconnected-(U1-GPIO31-Pad39) -> GPIO31
- U1 pad 40: unconnected-(U1-GPIO32-Pad40) -> GPIO32
- U1 pad 42: unconnected-(U1-GPIO33-Pad42) -> GPIO33
- U1 pad 43: unconnected-(U1-GPIO34-Pad43) -> GPIO34
- U1 pad 44: unconnected-(U1-GPIO35-Pad44) -> GPIO35
- U1 pad 45: unconnected-(U1-GPIO36-Pad45) -> SINTA
- U1 pad 46: unconnected-(U1-GPIO37-Pad46) -> SINTB
- U1 pad 47: unconnected-(U1-GPIO38-Pad47) -> UINTA
- U1 pad 48: unconnected-(U1-GPIO39-Pad48) -> UINTB
- U1 pad 49: unconnected-(U1-GPIO40_ADC0-Pad49) -> SDA
- U1 pad 52: unconnected-(U1-GPIO41_ADC1-Pad52) -> SCL
- U1 pad 58: unconnected-(U1-GPIO47_ADC7-Pad58) -> GPIO47
- U1 pad 80: unconnected-(U1-GPIO3-Pad80) -> LED0
